File: ethernetphy.kicad_sch (KiCad schematic)
At the start: 0 parts

Commit message: Add power sheet and update schematic connections
Added a new power sheet to the project and updated the main schematic to include connections for power, MCU, peripherals, and Ethernet PHY. Also added backup files and updated the Ethernet PHY schematic with symbol definitions and pin mappings.
Parts:
- added C15, C16: 32pF, symbol Device:C
- added C17: 0.01uF, symbol Device:C
- added C18, C20, C22, C24: 1uF, symbol Device:C
- added C19, C23: 0.1uF, symbol Device:C
- added C21, C25: 10uF, symbol Device:C
- added D4: LED, symbol Device:LED
- added JP1: Jumper_3_Open, symbol Jumper:Jumper_3_Open
- added R5: 100, symbol Device:R
- added R6: 6.49k, symbol Device:R
- added R7: 2.2k, symbol Device:R
- added S3: SKRPABE010, SKRPABE010:SW_SKRPABE010, symbol SKRPABE010:SKRPABE010
- added U2: DP83825IRMQT, DP83825IRMQT:XCVR_DP83825IRMQT, symbol DP83825IRMQT:DP83825IRMQT
- added Y2: ABM8-25.000MHZ-20-D1X-T, Crystal:Crystal_SMD_Abracon_ABM8G-4Pin_3.2x2.5mm, symbol MyLibrary:ABM8-25.000MHZ-20-D1X-T
Connections:
- new net: R7.1, S3.3, S3.4
- new net: R6.1, U2.14 (RBIAS)
- new net: D4.2 (A), R5.2
- new net +3V3: C18.1, C19.1, C20.1, C21.1, JP1.3 (B), U2.6 (VDDA3V3)
- new net +3V3IO: C22.1, C23.1, C24.1, C25.1, U2.19 (VDDIO)
- new net ETH_RD_M: U2.7 (RD_M)
- new net ETH_RD_P: U2.8 (RD_P)
- new net ETH_TD_M: U2.10 (TD_M)
- new net ETH_TD_P: U2.11 (TD_P)
- new net GND: C15.2, C16.2, C17.2, C18.2, C19.2, C20.2, C21.2, C22.2, C23.2, C24.2, C25.2, JP1.1 (A), R6.2, R7.2, U2.21 (GND__1), U2.25 (EXP), U2.26 (EXP__1), U2.27 (EXP__2), U2.28 (EXP__3), U2.29 (EXP__4), U2.30 (EXP__5), U2.9 (GND), Y2.2 (GND), Y2.4 (GND)
- new net LED0: R5.1, U2.4 (LED0/S(ANEG_DIS))
- new net PHY_MDC: U2.16 (MDC)
- new net PHY_MDIO: U2.15 (MDIO)
- new net PWDN: U2.3 (INTR/PWRDN)
- new net RMII_CLK: U2.2 (50MHZOUT/LED2/S(RX_DV_EN))
- new net RMII_CRS_DV: U2.20 (CRS_DV/S(PHYADD1))
- new net RMII_RXD0: U2.18 (RX_D0/S(PHYADD0))
- new net RMII_RXD1: U2.17 (RX_D1/S(MASTER/SLAVE))
- new net RMII_TXD0: U2.23 (TX_D0)
- new net RMII_TXD1: U2.24 (TX_D1)
- new net RMII_TX_EN: U2.1 (TX_EN)
- new net RST: C17.1, S3.1, S3.2, U2.5 (~{RST})
- new net RX_ER: JP1.2 (C), U2.22 (RX_ER/S(A-MDIX))
- new net XIN: C15.1, U2.13 (XI/50MHZIN), Y2.3 (OUT)
- new net XOUT: C16.1, U2.12 (XO), Y2.1 (EN)

Commit message: Update schematic power symbols and add backups
Replaced +48V and -48V power symbols with VDD and VSS in peripherals.kicad_sch, updated title blocks and paper sizes in all .kicad_sch files, and added new schematic symbols for test points, capacitors, resistors, MOSFET, and optocoupler in power.kicad_sch. Added multiple new backup ZIP files for POETempSensor.
Other:
- title: (none) -> Ethernet PHY
Changed lines of the file:
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@@
 	(generator_version "9.0")
 	(paper "A4")
+	(title_block
+		(title "Ethernet PHY")
+		(date "2025-11-09")
+		(rev "v0.1")
+	)
 	(junction
 		(at 181.61 109.22)
